File: Hardware/ATSAMD21G18A_Breakout.sch (EAGLE design)
At the start: 35 parts, among them J2 GRPB052VWVN-RC, J3 MF-CON-2.54mm-01x14, J4 MF-CON-2.54mm-01x14, J5 MF-CON-2.54mm-01x06, J6 MF-CON-2.54mm-01x06, SW1 MF-SW-TACT-4.2MM, U1 ATSAMD21G18A, U2 IP4234CZ6,125, U3 BQ24165RGET, U4 MF-REG-SOT235-3.3V-300mA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

Commit message: removed tag connect and added LDK320AM33R for the LDO
Parts:
- removed TC1: TC2030-IDC-NL, MF_Connectors:CON_02X03_SWD2TC_TC2030-IDC-NL
- U4: value MF-REG-SOT235-3.3V-300mA -> LDK320AM33R; HOUSEPART (none) -> No; MPN (none) -> LDK320AM33R
Connections:
- removed net SWO: TC1.PIN5
- net !RESET: no longer TC1.PIN6
- net 3.3V: no longer TC1.PIN1
- net GND: no longer TC1.PIN2
- net SWCLK: no longer TC1.PIN4
- net SWDIO: no longer TC1.PIN3
Changed lines of the file:
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@@
 <attribute name="MPN" value="ERJ-3EKF5101V"/>
 </part>
-<part name="U4" library="MF_IC_Power" deviceset="TLV702" device="33PDBVR" value="MF-REG-SOT235-3.3V-300mA"/>
-<part name="TC1" library="MF_Connectors" deviceset="CON_02X03" device="_TC2030-IDC-NL" technology="_SWD2TC" value="TC2030-IDC-NL"/>
-<part name="U$29" library="MF_Aesthetics" deviceset="POWER_RAIL" device="" value="3.3V"/>
-<part name="U$30" library="MF_Aesthetics" deviceset="GND_RAIL" device=""/>
+<part name="U4" library="MF_IC_Power" deviceset="TLV702" device="33PDBVR" value="LDK320AM33R">
+<attribute name="HOUSEPART" value="No"/>
+<attribute name="MPN" value="LDK320AM33R"/>
+<attribute name="URL" value=""/>
+</part>
 <part name="U3" library="PP_PowerIC" deviceset="BQ24165" device="RGET"/>
 <part name="X1" library="PP_FreqCtrl" deviceset="CRYSTAL" device="_FC-12M" value="FC-12M 32.7680KA-A3">
@@
 </part>
 <part name="U5" library="PP_DigitalIC" deviceset="DS1340Z" device="U-33+" value="DS1340U-33+T&amp;R">
-<attribute name="MPN" value="
-DS1340U-33+T&amp;R
-"/>
+<attribute name="MPN" value=" DS1340U-33+T&amp;R "/>
 </part>
 <part name="BATT1" library="PP_Connectors" deviceset="BATTERY" device="_KEYSTONE_1074"/>
@@
 <attribute name="NAME" x="123.19" y="22.86" size="1.016" layer="95" font="vector" align="top-left"/>
 <attribute name="VALUE" x="123.19" y="20.32" size="1.016" layer="96" font="vector"/>
-</instance>
-<instance part="TC1" gate="G$1" x="115.57" y="118.11" smashed="yes">
-<attribute name="LABEL01" x="123.19" y="118.11" size="1.016" layer="97" font="vector" rot="MR180" align="center-left"/>
-<attribute name="NAME" x="115.57" y="123.19" size="1.016" layer="95" font="vector" align="top-left"/>
-<attribute name="VALUE" x="115.57" y="120.65" size="1.016" layer="96" font="vector"/>
-<attribute name="LABEL02" x="138.43" y="118.11" size="1.016" layer="97" font="vector" rot="MR0" align="center-left"/>
-<attribute name="LABEL03" x="123.19" y="115.57" size="1.016" layer="97" font="vector" rot="MR180" align="center-left"/>
-<attribute name="LABEL04" x="138.43" y="115.57" size="1.016" layer="97" font="vector" rot="MR0" align="center-left"/>
-<attribute name="LABEL05" x="123.19" y="113.03" size="1.016" layer="97" font="vector" rot="MR180" align="center-left"/>
-<attribute name="LABEL06" x="138.43" y="113.03" size="1.016" layer="97" font="vector" rot="MR0" align="center-left"/>
-</instance>
-<instance part="U$29" gate="G$1" x="104.14" y="123.19" smashed="yes" rot="MR0">
-<attribute name="VALUE" x="104.14" y="125.73" size="1.016" layer="96" font="vector" rot="MR0" align="center"/>
-</instance>
-<instance part="U$30" gate="G$1" x="160.02" y="106.68" smashed="yes" rot="MR0">
-<attribute name="VALUE" x="160.02" y="104.14" size="1.016" layer="96" font="vector" rot="MR180" align="center"/>
 </instance>
 <instance part="U3" gate="G$1" x="-81.28" y="58.42" smashed="yes">
@@
 <label x="208.28" y="11.43" size="1.016" layer="95" font="vector" rot="R180" xref="yes"/>
 </segment>
-<segment>
-<pinref part="TC1" gate="G$1" pin="PIN2"/>
-<pinref part="U$30" gate="G$1" pin="P$1"/>
-<wire x1="148.59" y1="118.11" x2="160.02" y2="118.11" width="0.1524" layer="91"/>
-<wire x1="160.02" y1="118.11" x2="160.02" y2="109.22" width="0.1524" layer="91"/>
-</segment>
 </net>
 <net name="VDDCORE" class="0">
@@
 <label x="208.28" y="13.97" size="1.016" layer="95" font="vector" rot="R180" xref="yes"/>
 </segment>
-<segment>
-<pinref part="TC1" gate="G$1" pin="PIN1"/>
-<pinref part="U$29" gate="G$1" pin="P$1"/>
-<wire x1="113.03" y1="118.11" x2="104.14" y2="118.11" width="0.1524" layer="91"/>
-<wire x1="104.14" y1="118.11" x2="104.14" y2="120.65" width="0.1524" layer="91"/>
-</segment>
 </net>
 <net name="XIN32" class="0">
@@
 <wire x1="-5.08" y1="76.2" x2="-8.89" y2="76.2" width="0.1524" layer="91"/>
 <label x="-8.89" y="76.2" size="1.016" layer="95" font="vector" rot="R180" xref="yes"/>
-</segment>
-<segment>
-<pinref part="TC1" gate="G$1" pin="PIN6"/>
-<wire x1="148.59" y1="113.03" x2="151.13" y2="113.03" width="0.1524" layer="91"/>
-<label x="151.13" y="113.03" size="1.016" layer="95" font="vector" xref="yes"/>
 </segment>
 </net>
@@
 <label x="66.04" y="43.18" size="1.016" layer="95" font="vector" xref="yes"/>
 </segment>
-<segment>
-<pinref part="TC1" gate="G$1" pin="PIN3"/>
-<wire x1="113.03" y1="115.57" x2="110.49" y2="115.57" width="0.1524" layer="91"/>
-<label x="110.49" y="115.57" size="1.016" layer="95" font="vector" rot="R180" xref="yes"/>
-</segment>
 </net>
 <net name="SWCLK" class="0">
@@
 <wire x1="55.88" y1="45.72" x2="66.04" y2="45.72" width="0.1524" layer="91"/>
 <label x="66.04" y="45.72" size="1.016" layer="95" font="vector" xref="yes"/>
-</segment>
-<segment>
-<pinref part="TC1" gate="G$1" pin="PIN4"/>
-<wire x1="148.59" y1="115.57" x2="151.13" y2="115.57" width="0.1524" layer="91"/>
-<label x="151.13" y="115.57" size="1.016" layer="95" font="vector" xref="yes"/>
 </segment>
 </net>
@@
 </segment>
 </net>
-<net name="SWO" class="0">
-<segment>
-<pinref part="TC1" gate="G$1" pin="PIN5"/>
-<wire x1="113.03" y1="113.03" x2="110.49" y2="113.03" width="0.1524" layer="91"/>
-<label x="110.49" y="113.03" size="1.016" layer="95" font="vector" rot="R180" xref="yes"/>
-</segment>
-</net>
